File: can-node.kicad_sch (KiCad schematic)
At the start: 38 parts, among them J1 Conn_01x02_Pin, J10 Conn_01x06_Pin, J13 Conn_01x01_Socket, J14 Conn_01x01_Socket, J15 Conn_01x03_Pin, J16 Conn_01x02_Pin, J17 Conn_01x02_Pin, J2 Conn_01x02_Pin, J3 RJ45, J4 RJ45, J5 Conn_01x10_Pin, J6 Conn_01x04_Pin, J7 Conn_01x02_Pin, J8 Conn_01x01_Socket, J9 Conn_01x01_Socket, SW1 SW_DIP_x04, U1 ESP32-DEVKIT-V1

Commit message: routing attempt
Parts:
- removed R13: 60, Resistor_THT:R_Axial_DIN0204_L3.6mm_D1.6mm_P5.08mm_Horizontal, symbol Device:R
- added J11: Conn_01x02_Socket, Connector_Wire:SolderWire-0.1sqmm_1x02_P3.6mm_D0.4mm_OD1mm, symbol Connector:Conn_01x02_Socket
Connections:
- net CAN+: now also J11.1 (Pin_1)
- net CAN-: now also J11.2 (Pin_2)
- net DIR: now also U1.23 (D25); no longer U1.24 (D26)
- net ENC-A: now also U1.19 (D34); no longer U1.22 (D33)
- net ENC-B: now also U1.22 (D33); no longer U1.19 (D34)
- net FSYNC: now also U1.9 (D18); no longer U1.10 (D19)
- net INT: now also U1.10 (D19); no longer U1.9 (D18)
- net LED0: now also R9.2; no longer R3.2
- net LED1: now also R10.2; no longer R8.2
- net LED2: now also R8.2; no longer R9.2
- net LED3: now also R3.2; no longer R10.2
- net PWM: now also U1.24 (D26); no longer U1.23 (D25)
Changed lines of the file:
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@@
+    (stroke (width 0) (type default))
+  )
+  (wire (pts (xy 67.31 138.43) (xy 71.12 138.43))
     (stroke (width 0) (type default))
   )
@@
     (stroke (width 0) (type default))
   )
-  (wire (pts (xy 71.12 130.81) (xy 86.36 130.81))
-    (stroke (width 0) (type default))
-  )
   (wire (pts (xy 33.02 71.12) (xy 35.56 71.12))
     (stroke (width 0) (type default))
@@
     (stroke (width 0) (type default))
   )
-  (wire (pts (xy 71.12 143.51) (xy 86.36 143.51))
-    (stroke (width 0) (type default))
-  )
   (wire (pts (xy 111.76 45.72) (xy 111.76 60.96))
     (stroke (width 0) (type default))
@@
     (stroke (width 0) (type default))
   )
+  (wire (pts (xy 67.31 135.89) (xy 71.12 135.89))
+    (stroke (width 0) (type default))
+  )
   (wire (pts (xy 66.04 63.5) (xy 68.58 63.5))
     (stroke (width 0) (type default))
@@
     (stroke (width 0) (type default))
   )
-  (wire (pts (xy 86.36 133.35) (xy 86.36 130.81))
-    (stroke (width 0) (type default))
-  )
   (wire (pts (xy 114.3 40.64) (xy 114.3 38.1))
     (stroke (width 0) (type default))
@@
   )
   (wire (pts (xy 33.02 68.58) (xy 35.56 68.58))
-    (stroke (width 0) (type default))
-  )
-  (wire (pts (xy 86.36 143.51) (xy 86.36 140.97))
     (stroke (width 0) (type default))
   )
@@
     )
   )
-  (global_label "PWM" (shape input) (at 68.58 58.42 0) (fields_autoplaced)
-    (effects (font (size 1.27 1.27)) (justify left))
-    (property "Intersheetrefs" "${INTERSHEET_REFS}" (at 75.738 58.42 0)
+  (global_label "DIR" (shape input) (at 68.58 58.42 0) (fields_autoplaced)
+    (effects (font (size 1.27 1.27)) (justify left))
+    (property "Intersheetrefs" "${INTERSHEET_REFS}" (at 74.71 58.42 0)
       (effects (font (size 1.27 1.27)) (justify left) hide)
     )
@@
     )
   )
-  (global_label "CAN-" (shape input) (at 71.12 143.51 180) (fields_autoplaced)
-    (effects (font (size 1.27 1.27)) (justify right))
-    (property "Intersheetrefs" "${INTERSHEET_REFS}" (at 62.8733 143.51 0)
-      (effects (font (size 1.27 1.27)) (justify right) hide)
-    )
-  )
-  (global_label "INT" (shape output) (at 33.02 71.12 180) (fields_autoplaced)
-    (effects (font (size 1.27 1.27)) (justify right))
-    (property "Intersheetrefs" "${INTERSHEET_REFS}" (at 27.1319 71.12 0)
+  (global_label "CAN-" (shape input) (at 67.31 138.43 180) (fields_autoplaced)
+    (effects (font (size 1.27 1.27)) (justify right))
+    (property "Intersheetrefs" "${INTERSHEET_REFS}" (at 59.0633 138.43 0)
+      (effects (font (size 1.27 1.27)) (justify right) hide)
+    )
+  )
+  (global_label "FSYNC" (shape output) (at 33.02 71.12 180) (fields_autoplaced)
+    (effects (font (size 1.27 1.27)) (justify right))
+    (property "Intersheetrefs" "${INTERSHEET_REFS}" (at 24.0476 71.12 0)
       (effects (font (size 1.27 1.27)) (justify right) hide)
     )
@@
     )
   )
-  (global_label "LED1" (shape output) (at 25.4 152.4 180) (fields_autoplaced)
+  (global_label "LED2" (shape output) (at 25.4 152.4 180) (fields_autoplaced)
     (effects (font (size 1.27 1.27)) (justify right))
     (property "Intersheetrefs" "${INTERSHEET_REFS}" (at 17.7582 152.4 0)
@@
     )
   )
-  (global_label "ENC-A" (shape output) (at 68.58 68.58 0) (fields_autoplaced)
-    (effects (font (size 1.27 1.27)) (justify left))
-    (property "Intersheetrefs" "${INTERSHEET_REFS}" (at 77.9757 68.58 0)
+  (global_label "ENC-B" (shape output) (at 68.58 68.58 0) (fields_autoplaced)
+    (effects (font (size 1.27 1.27)) (justify left))
+    (property "Intersheetrefs" "${INTERSHEET_REFS}" (at 78.1571 68.58 0)
       (effects (font (size 1.27 1.27)) (justify left) hide)
     )
@@
     )
   )
-  (global_label "ENC-B" (shape output) (at 68.58 73.66 0) (fields_autoplaced)
-    (effects (font (size 1.27 1.27)) (justify left))
-    (property "Intersheetrefs" "${INTERSHEET_REFS}" (at 78.1571 73.66 0)
+  (global_label "ENC-A" (shape output) (at 68.58 73.66 0) (fields_autoplaced)
+    (effects (font (size 1.27 1.27)) (justify left))
+    (property "Intersheetrefs" "${INTERSHEET_REFS}" (at 77.9757 73.66 0)
       (effects (font (size 1.27 1.27)) (justify left) hide)
     )
@@
     )
   )
-  (global_label "LED0" (shape output) (at 25.4 138.43 180) (fields_autoplaced)
+  (global_label "LED3" (shape output) (at 25.4 138.43 180) (fields_autoplaced)
     (effects (font (size 1.27 1.27)) (justify right))
     (property "Intersheetrefs" "${INTERSHEET_REFS}" (at 17.7582 138.43 0)
@@
     )
   )
-  (global_label "FSYNC" (shape output) (at 33.02 73.66 180) (fields_autoplaced)
-    (effects (font (size 1.27 1.27)) (justify right))
-    (property "Intersheetrefs" "${INTERSHEET_REFS}" (at 24.0476 73.66 0)
+  (global_label "INT" (shape output) (at 33.02 73.66 180) (fields_autoplaced)
+    (effects (font (size 1.27 1.27)) (justify right))
+    (property "Intersheetrefs" "${INTERSHEET_REFS}" (at 27.1319 73.66 0)
       (effects (font (size 1.27 1.27)) (justify right) hide)
     )
@@
     )
   )
-  (global_label "CAN+" (shape input) (at 71.12 130.81 180) (fields_autoplaced)
-    (effects (font (size 1.27 1.27)) (justify right))
-    (property "Intersheetrefs" "${INTERSHEET_REFS}" (at 62.8733 130.81 0)
+  (global_label "CAN+" (shape input) (at 67.31 135.89 180) (fields_autoplaced)
+    (effects (font (size 1.27 1.27)) (justify right))
+    (property "Intersheetrefs" "${INTERSHEET_REFS}" (at 59.0633 135.89 0)
       (effects (font (size 1.27 1.27)) (justify right) hide)
     )
@@
     )
   )
-  (global_label "LED2" (shape output) (at 25.4 166.37 180) (fields_autoplaced)
+  (global_label "LED0" (shape output) (at 25.4 166.37 180) (fields_autoplaced)
     (effects (font (size 1.27 1.27)) (justify right))
     (property "Intersheetrefs" "${INTERSHEET_REFS}" (at 17.7582 166.37 0)
@@
     )
   )
-  (global_label "LED3" (shape output) (at 25.4 180.34 180) (fields_autoplaced)
+  (global_label "LED1" (shape output) (at 25.4 180.34 180) (fields_autoplaced)
     (effects (font (size 1.27 1.27)) (justify right))
     (property "Intersheetrefs" "${INTERSHEET_REFS}" (at 17.7582 180.34 0)
@@
     )
   )
-  (global_label "DIR" (shape input) (at 68.58 60.96 0) (fields_autoplaced)
-    (effects (font (size 1.27 1.27)) (justify left))
-    (property "Intersheetrefs" "${INTERSHEET_REFS}" (at 74.71 60.96 0)
+  (global_label "PWM" (shape input) (at 68.58 60.96 0) (fields_autoplaced)
+    (effects (font (size 1.27 1.27)) (justify left))
+    (property "Intersheetrefs" "${INTERSHEET_REFS}" (at 75.738 60.96 0)
       (effects (font (size 1.27 1.27)) (justify left) hide)
     )
@@
         (path "/f336cf10-c71e-46f0-bc5d-32363ccffe11"
           (reference "D1") (unit 1)
-        )
-      )
-    )
-  )
-  (symbol (lib_id "Device:R") (at 86.36 137.16 0) (unit 1)
-    (in_bom yes) (on_board yes) (dnp no) (fields_autoplaced)
-    (property "Reference" "R13" (at 88.9 135.89 0)
-      (effects (font (size 1.27 1.27)) (justify left))
-    )
-    (property "Value" "60" (at 88.9 138.43 0)
-      (effects (font (size 1.27 1.27)) (justify left))
-    )
-    (property "Footprint" "Resistor_THT:R_Axial_DIN0204_L3.6mm_D1.6mm_P5.08mm_Horizontal" (at 84.582 137.16 90)
-      (effects (font (size 1.27 1.27)) hide)
-    )
-    (property "Datasheet" "~" (at 86.36 137.16 0)
-      (effects (font (size 1.27 1.27)) hide)
-    )
-    (pin "1")
-    (pin "2")
-    (instances
-      (project "can-node"
-        (path "/d1086eed-11fd-4182-90da-fa3935545562"
-          (reference "R13") (unit 1)
         )
       )
@@
         )
       )
+    )
+  )
+  (symbol (lib_id "Connector:Conn_01x02_Socket") (at 76.2 135.89 0) (unit 1)
+    (in_bom yes) (on_board yes) (dnp no) (fields_autoplaced)
+    (property "Reference" "J11" (at 77.47 135.89 0)
+      (effects (font (size 1.27 1.27)) (justify left))
+    )
+    (property "Value" "Conn_01x02_Socket" (at 77.47 138.43 0)
+      (effects (font (size 1.27 1.27)) (justify left))
+    )
+    (property "Footprint" "Connector_Wire:SolderWire-0.1sqmm_1x02_P3.6mm_D0.4mm_OD1mm" (at 76.2 135.89 0)
+      (effects (font (size 1.27 1.27)) hide)
+    )
+    (property "Datasheet" "~" (at 76.2 135.89 0)
+      (effects (font (size 1.27 1.27)) hide)
+    )
+    (pin "1")
+    (pin "2")
+    (instances
+      (project "can-node"
+        (path "/d1086eed-11fd-4182-90da-fa3935545562"
+          (reference "J11") (unit 1)
+        )
+      )

Commit message: update for 3D
Parts:
- J15: footprint Connector_JST:JST_PH_B3B-PH-K_1x03_P2.00mm_Vertical -> Connector_JST:JST_PH_S3B-PH-K_1x03_P2.00mm_Horizontal
Changed lines of the file:
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@@
     (effects (font (size 1.27 1.27)) (justify left bottom))
   )
-  (text "CAN Termination" (at 82.55 123.19 0)
+  (text "CAN Termination" (at 82.55 149.86 0)
     (effects (font (size 1.27 1.27)) (justify left bottom))
   )
@@
     (effects (font (size 1.27 1.27)) (justify left bottom))
   )
-  (text "CAN Debug" (at 87.63 149.86 0)
+  (text "CAN Debug" (at 87.63 121.92 0)
     (effects (font (size 1.27 1.27)) (justify left bottom))
   )
@@
       (effects (font (size 1.27 1.27)) (justify right))
     )
-    (property "Footprint" "Connector_JST:JST_PH_B3B-PH-K_1x03_P2.00mm_Vertical" (at 260.35 72.39 0)
-      (effects (font (size 1.27 1.27)) hide)
-    )
+    (property "Footprint" "Connector_JST:JST_PH_S3B-PH-K_1x03_P2.00mm_Horizontal" (at 260.35 72.39 0)
+      (effects (font (size 1.27 1.27)) hide)
+    )

Commit message: update with feedback
Parts:
- removed J16: Conn_01x02_Pin, Connector_Wire:SolderWire-1sqmm_1x02_P5.4mm_D1.4mm_OD2.7mm, symbol Connector:Conn_01x02_Pin
- removed J7: Conn_01x02_Pin, Connector_Wire:SolderWire-1.5sqmm_1x02_P7.8mm_D1.7mm_OD3.9mm, symbol Connector:Conn_01x02_Pin
- J17: footprint Connector_Wire:SolderWire-1sqmm_1x02_P5.4mm_D1.4mm_OD2.7mm -> Connector_Wire:SolderWire-1sqmm_1x02_P7.8mm_D1.4mm_OD3.9mm
Other:
- moved on the sheet: J1, J10, J15, J17, J2, J5, J6, R1, R2
