File: can-node.kicad_sch (KiCad schematic)
At the start: 36 parts, among them J1 Conn_01x02_Pin, J10 Conn_01x06_Pin, J11 Conn_01x02_Socket, J13 Conn_01x01_Socket, J14 Conn_01x01_Socket, J15 Conn_01x03_Pin, J17 Conn_01x02_Pin, J2 Conn_01x02_Pin, J3 RJ45, J4 RJ45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

Commit message: finish reroute
Parts:
- D1: value LED -> POWER
- D2: value LED -> STATUS
- D3: value LED -> IMU CALI
- D4: value LED -> CTX
- D5: value LED -> SYNC
- D6: value LED -> CRX
- J10: value Conn_01x06_Pin -> MCP2551
- J13: value Conn_01x01_Socket -> SDA
- J14: value Conn_01x01_Socket -> SCL
- J15: value Conn_01x03_Pin -> MD13 SIGNAL
- J17: value Conn_01x02_Pin -> MD13S PWR
- J3, J4: value RJ45 -> CAN
- J5: value Conn_01x10_Pin -> MPU9250
- J6: value Conn_01x04_Pin -> ENCODER
- J8: value Conn_01x01_Socket -> CRX
- J9: value Conn_01x01_Socket -> CTX
- SW1: value SW_DIP_x04 -> ADDRESS
Connections:
- net +5V: now also J6.4 (Pin_4); no longer J6.1 (Pin_1)
- net ENC-A: now also J6.2 (Pin_2); no longer J6.3 (Pin_3)
- net ENC-B: now also J6.1 (Pin_1); no longer J6.4 (Pin_4)
- net GND: now also J6.3 (Pin_3); no longer J6.2 (Pin_2)

Commit message: fix 5V for MCP
Connections:
- net +5VA is gone; now on net +5V: J10.1 (Pin_1)
Changed lines of the file:
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@@
     )
   )
-  (symbol (lib_id "power:+5VA") (at 175.26 63.5 0) (unit 1)
+  (symbol (lib_id "power:+5V") (at 175.26 63.5 0) (unit 1)
     (in_bom yes) (on_board yes) (dnp no) (fields_autoplaced)
     (property "Reference" "#PWR034" (at 175.26 67.31 0)
       (effects (font (size 1.27 1.27)) hide)
     )
-    (property "Value" "+5VA" (at 175.26 58.42 0)
+    (property "Value" "+5V" (at 175.26 59.944 0)
       (effects (font (size 1.27 1.27)))
     )

Commit message: add 5V
Parts:
- added F1: 800 mA, Fuse:Fuse_0805_2012Metric_Pad1.15x1.40mm_HandSolder, symbol Device:Fuse
Connections:
- net +5V: now also F1.2; no longer U2.3 (V_OUT)
- new net: F1.1, U2.3 (V_OUT)
Other:
- moved on the sheet: U2
Changed lines of the file:
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@@
   (junction (at 132.08 48.26) (diameter 0) (color 0 0 0 0)
   )
+  (junction (at 191.77 27.94) (diameter 0) (color 0 0 0 0)
+  )
   (junction (at 49.53 166.37) (diameter 0) (color 0 0 0 0)
   )
@@
   )
   (junction (at 92.71 38.1) (diameter 0) (color 0 0 0 0)
-  )
-  (junction (at 191.77 27.94) (diameter 0) (color 0 0 0 0)
   )
   (junction (at 92.71 40.64) (diameter 0) (color 0 0 0 0)
@@
     (stroke (width 0) (type default))
   )
-  (wire (pts (xy 165.1 27.94) (xy 168.91 27.94))
+  (wire (pts (xy 154.94 27.94) (xy 158.75 27.94))
     (stroke (width 0) (type default))
   )
@@
     (stroke (width 0) (type default))
   )
+  (wire (pts (xy 189.23 27.94) (xy 191.77 27.94))
+    (stroke (width 0) (type default))
+  )
   (wire (pts (xy 38.1 152.4) (xy 35.56 152.4))
     (stroke (width 0) (type default))
@@
     (stroke (width 0) (type default))
   )
-  (wire (pts (xy 189.23 34.29) (xy 191.77 34.29))
+  (wire (pts (xy 179.07 27.94) (xy 181.61 27.94))
+    (stroke (width 0) (type default))
+  )
+  (wire (pts (xy 179.07 34.29) (xy 181.61 34.29))
     (stroke (width 0) (type default))
   )
@@
     (stroke (width 0) (type default))
   )
-  (wire (pts (xy 191.77 34.29) (xy 191.77 39.37))
+  (wire (pts (xy 181.61 34.29) (xy 181.61 39.37))
     (stroke (width 0) (type default))
   )
@@
     (stroke (width 0) (type default))
   )
-  (wire (pts (xy 166.37 34.29) (xy 168.91 34.29))
+  (wire (pts (xy 156.21 34.29) (xy 158.75 34.29))
     (stroke (width 0) (type default))
   )
@@
     (stroke (width 0) (type default))
   )
-  (wire (pts (xy 189.23 27.94) (xy 191.77 27.94))
-    (stroke (width 0) (type default))
-  )
   (wire (pts (xy 205.74 91.44) (xy 215.9 91.44))
     (stroke (width 0) (type default))
@@
     (stroke (width 0) (type default))
   )
-  (wire (pts (xy 166.37 34.29) (xy 166.37 39.37))
+  (wire (pts (xy 156.21 34.29) (xy 156.21 39.37))
     (stroke (width 0) (type default))
   )
@@
     (fill (type none))
   )
-  (rectangle (start 154.94 13.97) (end 208.28 50.8)
+  (rectangle (start 140.97 13.97) (end 208.28 50.8)
     (stroke (width 0) (type default))
     (fill (type none))
@@
     )
   )
-  (global_label "+12 V" (shape input) (at 165.1 27.94 180) (fields_autoplaced)
-    (effects (font (size 1.27 1.27)) (justify right))
-    (property "Intersheetrefs" "${INTERSHEET_REFS}" (at 156.0672 27.94 0)
+  (global_label "+12 V" (shape input) (at 154.94 27.94 180) (fields_autoplaced)
+    (effects (font (size 1.27 1.27)) (justify right))
+    (property "Intersheetrefs" "${INTERSHEET_REFS}" (at 145.9072 27.94 0)
       (effects (font (size 1.27 1.27)) (justify right) hide)
     )
@@
         (path "/d1086eed-11fd-4182-90da-fa3935545562"
           (reference "#FLG04") (unit 1)
+        )
+      )
+    )
+  )
+  (symbol (lib_id "Device:Fuse") (at 185.42 27.94 90) (unit 1)
+    (in_bom yes) (on_board yes) (dnp no) (fields_autoplaced)
+    (property "Reference" "F1" (at 185.42 22.86 90)
+      (effects (font (size 1.27 1.27)))
+    )
+    (property "Value" "800 mA" (at 185.42 25.4 90)
+      (effects (font (size 1.27 1.27)))
+    )
+    (property "Footprint" "Fuse:Fuse_0805_2012Metric_Pad1.15x1.40mm_HandSolder" (at 185.42 29.718 90)
+      (effects (font (size 1.27 1.27)) hide)
+    )
+    (property "Datasheet" "~" (at 185.42 27.94 0)
+      (effects (font (size 1.27 1.27)) hide)
+    )
+    (pin "1")
+    (pin "2")
+    (instances
+      (project "can-node"
+        (path "/d1086eed-11fd-4182-90da-fa3935545562"
+          (reference "F1") (unit 1)
         )
       )
@@
     )
   )
-  (symbol (lib_id "power:GND") (at 191.77 39.37 0) (unit 1)
-    (in_bom yes) (on_board yes) (dnp no) (fields_autoplaced)
-    (property "Reference" "#PWR012" (at 191.77 45.72 0)
-      (effects (font (size 1.27 1.27)) hide)
-    )
-    (property "Value" "GND" (at 191.77 44.45 0)
-      (effects (font (size 1.27 1.27)))
-    )
-    (property "Footprint" "" (at 191.77 39.37 0)
-      (effects (font (size 1.27 1.27)) hide)
-    )
-    (property "Datasheet" "" (at 191.77 39.37 0)
+  (symbol (lib_id "power:GND") (at 181.61 39.37 0) (unit 1)
+    (in_bom yes) (on_board yes) (dnp no) (fields_autoplaced)
+    (property "Reference" "#PWR012" (at 181.61 45.72 0)
+      (effects (font (size 1.27 1.27)) hide)
+    )
+    (property "Value" "GND" (at 181.61 44.45 0)
+      (effects (font (size 1.27 1.27)))
+    )
+    (property "Footprint" "" (at 181.61 39.37 0)
+      (effects (font (size 1.27 1.27)) hide)
+    )
+    (property "Datasheet" "" (at 181.61 39.37 0)
       (effects (font (size 1.27 1.27)) hide)
     )
@@
     )
   )
-  (symbol (lib_id "MINI360-buck:MINI360_Buck") (at 179.07 31.75 0) (unit 1)
-    (in_bom yes) (on_board yes) (dnp no) (fields_autoplaced)
-    (property "Reference" "U2" (at 179.07 21.59 0)
-      (effects (font (size 1.27 1.27)))
-    )
-    (property "Value" "~" (at 179.07 31.75 0)
-      (effects (font (size 1.27 1.27)))
-    )
-    (property "Footprint" "MINI_360_Buck:MINI_360_Buck" (at 180.34 39.37 0)
-      (effects (font (size 1.27 1.27)) hide)
-    )
-    (property "Datasheet" "" (at 179.07 31.75 0)
+  (symbol (lib_id "MINI360-buck:MINI360_Buck") (at 168.91 31.75 0) (unit 1)
+    (in_bom yes) (on_board yes) (dnp no) (fields_autoplaced)
+    (property "Reference" "U2" (at 168.91 21.59 0)
+      (effects (font (size 1.27 1.27)))
+    )
+    (property "Value" "~" (at 168.91 31.75 0)
+      (effects (font (size 1.27 1.27)))
+    )
+    (property "Footprint" "MINI_360_Buck:MINI_360_Buck" (at 170.18 39.37 0)
+      (effects (font (size 1.27 1.27)) hide)
+    )
+    (property "Datasheet" "" (at 168.91 31.75 0)
       (effects (font (size 1.27 1.27)) hide)
     )
@@
     )
   )
-  (symbol (lib_id "power:GND") (at 166.37 39.37 0) (unit 1)
-    (in_bom yes) (on_board yes) (dnp no) (fields_autoplaced)
-    (property "Reference" "#PWR019" (at 166.37 45.72 0)
-      (effects (font (size 1.27 1.27)) hide)
-    )
-    (property "Value" "GND" (at 166.37 44.45 0)
-      (effects (font (size 1.27 1.27)))
-    )
-    (property "Footprint" "" (at 166.37 39.37 0)
-      (effects (font (size 1.27 1.27)) hide)
-    )
-    (property "Datasheet" "" (at 166.37 39.37 0)
-      (effects (font (size 1.27 1.27)) hide)
-    )
+  (symbol (lib_id "power:GND") (at 156.21 39.37 0) (unit 1)
+    (in_bom yes) (on_board yes) (dnp no) (fields_autoplaced)
+    (property "Reference" "#PWR019" (at 156.21 45.72 0)
+      (effects (font (size 1.27 1.27)) hide)
+    )
+    (property "Value" "GND" (at 156.21 44.45 0)
+      (effects (font (size 1.27 1.27)))
+    )
+    (property "Footprint" "" (at 156.21 39.37 0)
+      (effects (font (size 1.27 1.27)) hide)
+    )
+    (property "Datasheet" "" (at 156.21 39.37 0)
+      (effects (font (size 1.27 1.27)) hide)
+    )

Commit message: rm i2c pull-ups
Parts:
- removed R1, R2: 4.7k, Resistor_THT:R_Axial_DIN0204_L3.6mm_D1.6mm_P5.08mm_Horizontal, symbol Device:R
Other:
- note removed: "I2C Pull-up"
Changed lines of the file:
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@@
   (junction (at 132.08 35.56) (diameter 0) (color 0 0 0 0)
-  )
-  (junction (at 148.59 176.53) (diameter 0) (color 0 0 0 0)
   )
   (junction (at 114.3 48.26) (diameter 0) (color 0 0 0 0)
@@
     (stroke (width 0) (type default))
   )
-  (wire (pts (xy 148.59 176.53) (xy 148.59 189.23))
-    (stroke (width 0) (type default))
-  )
   (wire (pts (xy 25.4 43.18) (xy 25.4 44.45))
     (stroke (width 0) (type default))
@@
     (stroke (width 0) (type default))
   )
-  (wire (pts (xy 158.75 189.23) (xy 160.02 189.23))
-    (stroke (width 0) (type default))
-  )
   (wire (pts (xy 25.4 152.4) (xy 27.94 152.4))
     (stroke (width 0) (type default))
@@
     (stroke (width 0) (type default))
   )
-  (wire (pts (xy 158.75 176.53) (xy 160.02 176.53))
-    (stroke (width 0) (type default))
-  )
   (wire (pts (xy 124.46 177.8) (xy 128.27 177.8))
     (stroke (width 0) (type default))
@@
     (stroke (width 0) (type default))
   )
-  (wire (pts (xy 148.59 189.23) (xy 151.13 189.23))
-    (stroke (width 0) (type default))
-  )
   (wire (pts (xy 111.76 25.4) (xy 111.76 22.86))
     (stroke (width 0) (type default))
@@
     (stroke (width 0) (type default))
   )
-  (wire (pts (xy 148.59 176.53) (xy 151.13 176.53))
-    (stroke (width 0) (type default))
-  )
   (wire (pts (xy 107.95 40.64) (xy 114.3 40.64))
     (stroke (width 0) (type default))
@@
     (stroke (width 0) (type default))
   )
-  (wire (pts (xy 148.59 170.18) (xy 148.59 176.53))
-    (stroke (width 0) (type default))
-  )
   (wire (pts (xy 33.02 55.88) (xy 35.56 55.88))
     (stroke (width 0) (type default))
@@
   )
   (rectangle (start 140.97 54.61) (end 186.69 87.63)
-    (stroke (width 0) (type default))
-    (fill (type none))
-  )
-  (rectangle (start 143.51 162.56) (end 172.72 194.31)
     (stroke (width 0) (type default))
     (fill (type none))
@@
     (effects (font (size 1.27 1.27)) (justify left bottom))
   )
-  (text "I2C Pull-up" (at 160.02 194.31 0)
-    (effects (font (size 1.27 1.27)) (justify left bottom))
-  )
   (text "12V to 5V Buck" (at 191.77 50.8 0)
     (effects (font (size 1.27 1.27)) (justify left bottom))
@@
     )
   )
-  (global_label "I2C-SCL" (shape input) (at 160.02 176.53 0) (fields_autoplaced)
-    (effects (font (size 1.27 1.27)) (justify left))
-    (property "Intersheetrefs" "${INTERSHEET_REFS}" (at 171.1695 176.53 0)
-      (effects (font (size 1.27 1.27)) (justify left) hide)
-    )
-  )
   (global_label "ADD1" (shape output) (at 120.65 38.1 0) (fields_autoplaced)
     (effects (font (size 1.27 1.27)) (justify left))
@@
     (property "Intersheetrefs" "${INTERSHEET_REFS}" (at 210.82 80.1528 90)
       (effects (font (size 1.27 1.27)) (justify right) hide)
-    )
-  )
-  (global_label "I2C-SDA" (shape input) (at 160.02 189.23 0) (fields_autoplaced)
-    (effects (font (size 1.27 1.27)) (justify left))
-    (property "Intersheetrefs" "${INTERSHEET_REFS}" (at 171.23 189.23 0)
-      (effects (font (size 1.27 1.27)) (justify left) hide)
     )
   )
@@
     )
   )
-  (symbol (lib_id "power:+3.3V") (at 148.59 170.18 0) (unit 1)
-    (in_bom yes) (on_board yes) (dnp no) (fields_autoplaced)
-    (property "Reference" "#PWR015" (at 148.59 173.99 0)
-      (effects (font (size 1.27 1.27)) hide)
-    )
-    (property "Value" "+3.3V" (at 148.59 165.1 0)
-      (effects (font (size 1.27 1.27)))
-    )
-    (property "Footprint" "" (at 148.59 170.18 0)
-      (effects (font (size 1.27 1.27)) hide)
-    )
-    (property "Datasheet" "" (at 148.59 170.18 0)
-      (effects (font (size 1.27 1.27)) hide)
-    )
-    (pin "1")
-    (instances
-      (project "can-node"
-        (path "/d1086eed-11fd-4182-90da-fa3935545562"
-          (reference "#PWR015") (unit 1)
-        )
-      )
-    )
-  )
   (symbol (lib_id "power:+5V") (at 20.32 106.68 0) (unit 1)
     (in_bom yes) (on_board yes) (dnp no) (fields_autoplaced)
@@
         (path "/d1086eed-11fd-4182-90da-fa3935545562"
           (reference "#PWR05") (unit 1)
-        )
-      )
-    )
-  )
-  (symbol (lib_id "Device:R") (at 154.94 176.53 90) (unit 1)
-    (in_bom yes) (on_board yes) (dnp no) (fields_autoplaced)
-    (property "Reference" "R1" (at 154.94 170.18 90)
-      (effects (font (size 1.27 1.27)))
-    )
-    (property "Value" "4.7k" (at 154.94 172.72 90)
-      (effects (font (size 1.27 1.27)))
-    )
-    (property "Footprint" "Resistor_THT:R_Axial_DIN0204_L3.6mm_D1.6mm_P5.08mm_Horizontal" (at 154.94 178.308 90)
-      (effects (font (size 1.27 1.27)) hide)
-    )
-    (property "Datasheet" "~" (at 154.94 176.53 0)
-      (effects (font (size 1.27 1.27)) hide)
-    )
-    (pin "1")
-    (pin "2")
-    (instances
-      (project "can-node"
-        (path "/d1086eed-11fd-4182-90da-fa3935545562"
-          (reference "R1") (unit 1)
         )
       )
@@
         )
       )
-    )
-  )
-  (symbol (lib_id "Device:R") (at 154.94 189.23 90) (unit 1)
-    (in_bom yes) (on_board yes) (dnp no) (fields_autoplaced)
-    (property "Reference" "R2" (at 154.94 182.88 90)
-      (effects (font (size 1.27 1.27)))
-    )
-    (property "Value" "4.7k" (at 154.94 185.42 90)
-      (effects (font (size 1.27 1.27)))
-    )
-    (property "Footprint" "Resistor_THT:R_Axial_DIN0204_L3.6mm_D1.6mm_P5.08mm_Horizontal" (at 154.94 191.008 90)
-      (effects (font (size 1.27 1.27)) hide)
-    )
-    (property "Datasheet" "~" (at 154.94 189.23 0)
-      (effects (font (size 1.27 1.27)) hide)
-    )
-    (pin "1")
-    (pin "2")
-    (instances
-      (project "can-node"
-        (path "/d1086eed-11fd-4182-90da-fa3935545562"
-          (reference "R2") (unit 1)
-        )
-      )
